File: PCB/NeopixelRGBVisualizer-Single.brd (EAGLE design)
At the start: 26.8 x 29.6 mm, 19 parts, among them IC1 MSGEQ7, Q1 16MHz, X1 STEREOJACK, X2 1751251

Commit message: Version of board sent out for prototyping.  Can connect with avrdude, having some other issues.
Parts:
- moved X2 4.00 mm to (6.50, 29.9)
- moved C7 2.50 mm to (3.25, 11.8), turned to 0 degrees
- moved U$1 1.75 mm to (6.75, 23.6)
- moved C3 0.50 mm to (7.25, 11.8), turned to 180 degrees
Routing:
- net N$1: track 8.67 -> 15.6 mm
- net GND: track 6.26 -> 0.00 mm
- net N$8: track 37.1 -> 32.8 mm
- net VIN: track 40.5 -> 44.5 mm
- net N$15: track 17.1 -> 13.4 mm
- net N$2: track 7.73 -> 11.1 mm
- net VCC: track 53.4 -> 50.4 mm
- net N$7: track 12.2 -> 14.5 mm
- net N$4: track 7.12 -> 5.47 mm
- net N$17: track 2.96 -> 4.51 mm
- net N$9: track 14.5 -> 13.6 mm
Other:
- board size 26.8 x 29.6 mm -> 26.8 x 33.6 mm
